Commit message: Fixes for the migration to melodic

File: urdf/xacros/rover_body.xacro (robot description, xacro)
@@ -5,7 +5,7 @@
 		<xacro:property name="body_config" value="${load_yaml (filename)}"/>
 		<!-- Define world link-->
-		<link name="world"/>
+		<link name="${name}_base_link"/>
 		<!-- Define rover base link-->
-		<link name="${name}_base_link">
+		<link name="${name}_base_link_dummy">
 			<inertial>
 				<xacro:property name="data" value="${body_config['body']['inertial']}"/>
@@ -41,6 +41,6 @@
 		<joint name="${name}_world_joint" type="${body_config['joint']['type']}">
 			<xacro:property name="tmp" value="${body_config['joint']['origin']}"/>
-			<parent link="world"/>
-			<child link="${name}_base_link"/>
+			<parent link="${name}_base_link"/>
+			<child link="${name}_base_link_dummy"/>
 			<origin xyz="${tmp['position']['x']} ${tmp['position']['y']} ${tmp['position']['z']}"
 			rpy="${tmp['orientation']['roll']} ${tmp['orientation']['pitch']} ${tmp['orientation']['yaw']}"/>

File: urdf/xacros/wheel_hub.xacro (robot description, xacro)
@@ -19,5 +19,5 @@
             <origin xyz="${reflect1*tmp['origin']['position']['x']} ${reflect2*tmp['origin']['position']['y']} ${tmp['origin']['position']['z']}"
                 rpy="${tmp['origin']['orientation']['roll']} ${tmp['origin']['orientation']['pitch']} ${tmp['origin']['orientation']['yaw']+(reflect2 -1)*pi/2}"/>
-            <parent link="${name}_base_link"/>
+            <parent link="${name}_base_link_dummy"/>
             <child link="${name}_${side}_steer_link"/>
             <axis xyz="0 0 1"/>

Commit message: minor fixes

File: urdf/xacros/rover_body.xacro (robot description, xacro)
@@ -164,5 +164,5 @@
 			<parent link="${name}_base_link_dummy"/>
 			<child link="${name}_scan_link"/>
-			<origin xyz="0 0 0.13" rpy="0 0 0"/>
+			<origin xyz="0 0 0.13" rpy="0 ${pi / 18} 0"/>
 		</joint>
 		<!-- DEFINE HERE THE RASPBERRY PI CAMERA LINK -->

Commit message: updates

File: urdf/xacros/rover_body.xacro (robot description, xacro)
@@ -164,5 +164,5 @@
 			<parent link="${name}_base_link_dummy"/>
 			<child link="${name}_scan_link"/>
-			<origin xyz="0 0 0.13" rpy="0 ${pi / 18} 0"/>
+			<origin xyz="0 0 0.13" rpy="0 ${pi / 36} 0"/>
 		</joint>
 		<!-- DEFINE HERE THE RASPBERRY PI CAMERA LINK -->
