Commit message: Adding gravity component to imu

File: urdf/xacros/plugins.xacro (robot description, xacro)
@@ -17,10 +17,9 @@
             </plugin>
         </gazebo>
-        <gazebo>
+        <!-- <gazebo>
             <plugin name="${name}_kinematic_plugin" filename="libarchimede_kinematics_gazebo_ros_simulation_plugin.so"/>
-        </gazebo>
+        </gazebo> -->
         <gazebo>
             <plugin name="${name}_odometry_plugin" filename="libarchimede_odometry_gazebo_plugin.so">
-                <!-- <topics_ns>Archimede<topics_ns/> -->
                 <integrator>Trapezi</integrator>
                 <odomTopicName>Archimede/odom</odomTopicName>
@@ -36,9 +35,9 @@
                 <SensorStateTopicName>Archimede/sensor_state</SensorStateTopicName>
                 <OdomMode>position</OdomMode>
-                <skipFrames>10</skipFrames>
+                <skipFrames>1</skipFrames>
             </plugin>
         </gazebo>
         <!-- INCLUDE HERE PLUGIN FOR IMU -->
-        <gazebo>
+        <!-- <gazebo>
             <plugin name="imu_plugin" filename="libgazebo_ros_imu.so">
             <alwaysOn>true</alwaysOn>
@@ -48,5 +47,5 @@
             <serviceName>imu_service</serviceName>
             <gaussianNoise>0.0</gaussianNoise>
-            <updateRate>0</updateRate>
+            <updateRate>100</updateRate>
             <imu>
                 <noise>
@@ -67,6 +66,45 @@
             </imu>
             </plugin>
+        </gazebo> -->
+        <!-- Try with hector gazebo plugin hector_gazebo_ros_imu-->
+         <gazebo>
+            <plugin name="${name}_imu_sim" filename="libhector_gazebo_ros_imu.so">
+                <updateRate>100</updateRate>
+                <!-- <robotNamespace></robotNamespace> -->
+                <bodyName>${name}_imu_link</bodyName>
+                <frameId>${name}_imu_link</frameId>
+                <topicName>Archimede/imu</topicName>
+                <accelOffset>0 0 0</accelOffset>
+                <accelDrift>0 0 0</accelDrift>
+                <accelGaussianNoise>0 0 0</accelGaussianNoise>
+                <rateOffset>0 0 0</rateOffset>
+                <rateDrift>0 0 0</rateDrift>
+                <rateGaussianNoise>0 0 0</rateGaussianNoise>
+                <yawOffset>0</yawOffset>
+                <yawDrift>0</yawDrift>
+                <yawGaussianNoise>0</yawGaussianNoise>
+            </plugin>
         </gazebo>
-        <gazebo>
+        <!-- <gazebo reference="${name}_imu_link">
+            <gravity>true</gravity>
+            <sensor name="imu_sensor" type="imu">
+            <always_on>true</always_on>
+            <update_rate>100</update_rate>
+            <visualize>true</visualize>
+            <topic>__default_topic__</topic>
+            <plugin filename="libgazebo_ros_imu_sensor.so" name="imu_plugin">
+                <topicName>${name}/imu</topicName>
+                <bodyName>${name}_imu_link</bodyName>
+                <updateRateHZ>10.0</updateRateHZ>
+                <gaussianNoise>0.0</gaussianNoise>
+                <xyzOffset>0 0 0</xyzOffset>
+                <rpyOffset>0 0 0</rpyOffset>
+                <frameName>${name}_imu_link</frameName>
+                <initialOrientationAsReference>false</initialOrientationAsReference>
+            </plugin>
+            <pose>0 0 0 0 0 0</pose>
+            </sensor>
+        </gazebo>  -->
+        <!-- <gazebo>
             <plugin name="${name}_get_body_pose" filename="libarchimede_get_link_state.so">
                 <saveDir>$(find robot4ws_simulations)/data</saveDir>
@@ -83,5 +121,5 @@
                 <worldMode>false</worldMode>
             </plugin>
-        </gazebo>
+        </gazebo> -->
         <gazebo>
             <plugin name="${name}_magetic_sensor" filename="libhector_gazebo_ros_magnetic.so">

File: urdf/xacros/rover_body.xacro (robot description, xacro)
@@ -19,4 +19,15 @@
 		<!-- Define world link-->
 		<link name="${name}_base_link"/>
+		<!-- Define foot print-->
+		<!-- <link name="${name}_foot_print"/>
+		<joint name="${name}_foot_print_joint" type="fixed">
+			<parent link="${name}_base_link_dummy"/>
+			<child link="${name}_foot_print"/>
+			<origin xyz="0 0 -0.16" rpy="0 0 0"/>
+		</joint> -->
+		<!-- <gazebo reference="${name}_foot_print_joint">
+			<disableFixedJointLumping>true</disableFixedJointLumping>
+			<preserveFixedJoint>true</preserveFixedJoint>
+		</gazebo> -->
 		<!-- Define rover base link-->
 		<link name="${name}_base_link_dummy">
@@ -144,4 +155,8 @@
 			<origin xyz="0 0 0.08" rpy="0 0 0"/>
 		</joint>
+		<!-- <gazebo reference="${name}_imu_joint">
+			<disableFixedJointLumping>true</disableFixedJointLumping>
+			<preserveFixedJoint>true</preserveFixedJoint>
+		</gazebo>  -->
 		<!-- DEFINE HERE THE SCAN LINK -->
 		<link name="${name}_scan_link"/>

File: urdf/xacros/sensors.xacro (robot description, xacro)
@@ -84,5 +84,11 @@
             <sensor name="${name}_d435i_color" type="camera">
                 <camera name="${name}_d435i">
-                <horizontal_fov>1.2112585008840648</horizontal_fov>
+      <gazebo reference="${name}_imu_link">
+            <sensor type="imu" name="imu">
+            <always_on>true</always_on>
+            <visualize>$(arg visualize_imu)</visualize>
+            </sensor>
+            <material>Gazebo/Grey</material>
+        </gazebo>          <horizontal_fov>1.2112585008840648</horizontal_fov>
                 <image>
                     <width>1920</width>
@@ -130,5 +136,11 @@
                 <horizontal_fov>1.4870205226991688</horizontal_fov>
                 <image>
-                    <width>1280</width>
+                   <gazebo reference="${name}_imu_link">
+            <sensor type="imu" name="imu">
+            <always_on>true</always_on>
+            <visualize>$(arg visualize_imu)</visualize>
+            </sensor>
+            <material>Gazebo/Grey</material>
+        </gazebo> <width>1280</width>
                     <height>720</height>
                     <format>L_INT8</format>
@@ -139,5 +151,11 @@
                 </clip>
                 <noise>
-                    <type>gaussian</type>
+                   <gazebo reference="${name}_imu_link">
+            <sensor type="imu" name="imu">
+            <always_on>true</always_on>
+            <visualize>$(arg visualize_imu)</visualize>
+            </sensor>
+            <material>Gazebo/Grey</material>
+        </gazebo> <type>gaussian</type>
                     <mean>0.0</mean>
                     <stddev>0.05</stddev>
@@ -150,5 +168,11 @@
             <sensor name="${name}_d435i_depth" type="depth">
                 <camera name="${name}_d435i">
-                <horizontal_fov>1.4870205226991688</horizontal_fov>
+      <gazebo reference="${name}_imu_link">
+            <sensor type="imu" name="imu">
+            <always_on>true</always_on>
+            <visualize>$(arg visualize_imu)</visualize>
+            </sensor>
+            <material>Gazebo/Grey</material>
+        </gazebo>          <horizontal_fov>1.4870205226991688</horizontal_fov>
                 <image>
                     <width>1280</width>

Commit message: apply_PID_force_velocity plugin

File: urdf/xacros/plugins.xacro (robot description, xacro)
@@ -9,5 +9,5 @@
     <xacro:arg name="realsense_point_could" default="false"/>
     <!-- <xacro:arg name="" -->
-	<xacro:macro name="rover_plugins" params="name">
+	<xacro:macro name="rover_plugins" params="name include_terrain_slip_plugin">
         <gazebo>
             <plugin name="gazebo_ros_control" filename="libgazebo_ros_control.so">
@@ -123,5 +123,5 @@
         </gazebo> -->
         <gazebo>
-            <plugin name="${name}_magetic_sensor" filename="libhector_gazebo_ros_magnetic.so">
+            <plugin name="${name}_magnetic_sensor" filename="libhector_gazebo_ros_magnetic.so">
                 <updateRate>100</updateRate>
                 <robotNamespace>Archimede</robotNamespace>
@@ -130,4 +130,15 @@
             </plugin>
         </gazebo>
+        <xacro:if value="${include_terrain_slip_plugin}">
+            <gazebo>
+                <plugin name="archimede_apply_artificial_slip" filename="libarchimede_apply_artificial_slip.so">
+                    <apply_mode>force</apply_mode> <!-- force / velocity-->
+                    <pid_kp>2200</pid_kp>
+                    <pid_ki>2200000</pid_ki>
+                    <pid_kd>0</pid_kd>
+                    <pid_i_max>25</pid_i_max>
+                </plugin>
+            </gazebo>
+        </xacro:if>
 	</xacro:macro>
 </robot>

Commit message: update: add terramechanic plugin for all wheels

File: urdf/xacros/plugins.xacro (robot description, xacro)
@@ -143,7 +143,8 @@
         </xacro:if>
         <xacro:if value="${include_wheels_terramechanic_model}">
-            <xacro:property name="use_compact_model" value="true" /> <!-- true/false -->
+            <xacro:property name="use_compact_model" value="false" /> <!-- true/false -->
             <gazebo>
-                <plugin name="${name}_br_terramech_model" filename="libapply_single_wheel_terramechanic_model.so">
+                <!-- Single Terramechanics Model for Each Wheel -->
+                <!-- <plugin name="${name}_br_terramech_model" filename="libapply_single_wheel_terramechanic_model.so">
                     <link_name>Archimede_br_wheel_link</link_name>
                     <use_compact_model>${use_compact_model}</use_compact_model>
@@ -160,4 +161,8 @@
                     <link_name>Archimede_fl_wheel_link</link_name>
                     <use_compact_model>${use_compact_model}</use_compact_model>
+                </plugin> -->
+                <!-- Unified Terramechanics Model for All Wheels -->
+                <plugin name="${name}_terramech_model" filename="libapply_all_wheels_terramechanic_model.so">
+                    <use_compact_model>${use_compact_model}</use_compact_model>
                 </plugin>
             </gazebo>

Commit message: update: add ML plugin topic field & terramech passive option

File: urdf/xacros/plugins.xacro (robot description, xacro)
@@ -139,4 +139,7 @@
                     <pid_i_max>25</pid_i_max>
                     <last_input_vels_to_save>10</last_input_vels_to_save>
+                    <topic>ml_velocity_predictions</topic> <!-- topic with ML predictions -->
+                </plugin>
+                <plugin name="apply_soil_terrain" filename="libapply_soil_terrain.so">
                 </plugin>
             </gazebo>
@@ -144,4 +147,16 @@
         <xacro:if value="${include_wheels_terramechanic_model}">
             <xacro:property name="use_compact_model" value="false" /> <!-- true/false -->
+            <xacro:if value="${include_terrain_slip_plugin}">
+                <!-- if both plugin are active, the terramechanic one does not interact with gazebo (apply forces, modify frictions, ecc), but
+                    only publishes its results (confrontation purposes) -->
+                <xacro:property name="passive_plugin" value="true" />
+            </xacro:if>
+            <xacro:unless value="${include_terrain_slip_plugin}">
+                <xacro:property name="passive_plugin" value="false" />
+                <gazebo>
+                    <plugin name="apply_soil_terrain" filename="libapply_soil_terrain.so">
+                    </plugin>
+                </gazebo>
+            </xacro:unless>
             <gazebo>
                 <!-- Single Terramechanics Model for Each Wheel -->
@@ -165,4 +180,5 @@
                 <plugin name="${name}_terramech_model" filename="libapply_all_wheels_terramechanic_model.so">
                     <use_compact_model>${use_compact_model}</use_compact_model>
+                    <passive_plugin>${passive_plugin}</passive_plugin>
                 </plugin>
             </gazebo>
