Commit message: Full stable model

File: urdf/rover.urdf.xacro (robot description, xacro)
@@ -1,7 +1,18 @@
 <?xml version="1.0"?>
 <robot xmlns:xacro="http://www.ros.org/wiki/xacro" name="Archimede">
+	<xacro:arg name="include_plugins" default="true"/>
+	<xacro:arg name="include_kinematics_plugin" default="true"/>
+	<xacro:arg name="include_ros_control" default="true"/>
+	<xacro:arg name="realsense_use_nominal_extrinsics" default="true"/>
+	<!-- camera specific parameters -->
+	<xacro:arg name="topics_ns" default="Archimede"/>
+	<xacro:arg name="publish_pointcloud" default="true"/>
+	<xacro:arg name="add_plug" default="false"/>
 	<xacro:include filename="$(find robot4ws_description)/urdf/xacros/rover_body.xacro"/>
 	<xacro:include filename="$(find robot4ws_description)/urdf/xacros/wheel_hub.xacro"/>
 	<xacro:include filename="$(find robot4ws_description)/urdf/xacros/materials.xacro"/>
+	<xacro:include filename="$(find robot4ws_description)/urdf/xacros/plugins.xacro"/>
+	<xacro:include filename="$(find robot4ws_description)/urdf/xacros/sensors.xacro"/>
+	<xacro:include filename="$(find realsense2_description)/urdf/_d435i.urdf.xacro"/>
 	<!-- Include rover base -->
 	<xacro:rover_base name="Archimede">
@@ -19,3 +30,13 @@
 	<xacro:rover_wheel_hub name="Archimede" side="br" reflect1="-1" reflect2="-1">
 	</xacro:rover_wheel_hub>
+	<!-- INCLUDE REALSENSE D435I STEREOCAMERA -->
+	<xacro:sensor_d435i name="rs_d435i" topics_ns="$(arg topics_ns)" parent="Archimede_realsense_d435i_link" use_nominal_extrinsics="$(arg realsense_use_nominal_extrinsics)" publish_pointcloud="$(arg publish_pointcloud)" add_plug="$(arg add_plug)">
+		<origin xyz="0 0 0" rpy="0 0 0"/>
+	</xacro:sensor_d435i>
+	<!-- Include Sensors -->
+	<xacro:rover_sensors name="Archimede"/>
+	<!-- Include Rover Plugins -->
+	<xacro:if value="$(arg include_plugins)">
+		<xacro:rover_plugins name="Archimede"/>
+	</xacro:if>
 </robot>

File: urdf/xacros/rover_body.xacro (robot description, xacro)
@@ -38,4 +38,37 @@
 			</visual>
 		</link>
+		<!-- DEFINE HERE THE IMU LINK -->
+		<link name="${name}_imu_link"/>
+		<joint name="${name}_imu_joint" type="fixed">
+			<parent link="${name}_base_link_dummy"/>
+			<child link="${name}_imu_link"/>
+			<origin xyz="0 0 0.08" rpy="0 0 0"/>
+		</joint>
+		<!-- DEFINE HERE THE SCAN LINK -->
+		<link name="${name}_scan_link"/>
+		<joint name="${name}_scan_joint" type="fixed">
+			<parent link="${name}_base_link_dummy"/>
+			<child link="${name}_scan_link"/>
+			<origin xyz="0 0 0.13" rpy="0 0 0"/>
+		</joint>
+		<!-- DEFINE HERE THE RASPBERRY PI CAMERA LINK -->
+		<link name="${name}_pi_camera_link"/>
+		<joint name="${name}_pi_camera_joint" type="fixed">
+			<parent link="${name}_base_link_dummy"/>
+			<child link="${name}_pi_camera_link"/>
+			<origin xyz="0.15 0 0.075" rpy="0 0 0"/>
+		</joint>
+		<link name="${name}_pi_camera_color_optical_frame"/>
+		<joint name="${name}_pi_camera_color_optical_joint" type="fixed">
+			<parent link="${name}_pi_camera_link"/>
+			<child link="${name}_pi_camera_color_optical_frame"/>
+			<origin xyz="0 0 0.005" rpy="0 0 0"/>
+		</joint>
+		<link name="${name}_realsense_d435i_link"/>
+		<joint name="${name}_realsense_joint" type="fixed">
+			<parent link="${name}_base_link_dummy"/>
+			<child link="${name}_realsense_d435i_link"/>
+			<origin xyz="0.15 0 0.2" rpy="0 0 0"/>
+		</joint>
 		<!-- Define here the world joint -->
 		<joint name="${name}_world_joint" type="${body_config['joint']['type']}">

File: urdf/xacros/wheel_hub.xacro (robot description, xacro)
@@ -85,5 +85,5 @@
             <parent link="${name}_${side}_steer_link"/>
             <child link="${name}_${side}_wheel_link"/>
-            <axis xyz="0 0 1"/>
+            <axis xyz="0 1 0"/>
         </joint>
         <gazebo reference="${name}_${side}_wheel_link">
@@ -91,4 +91,22 @@
         </gazebo>
     <!-- Define here the transmission -->
+        <transmission name="${name}_${side}_drive_transmission}">
+            <type>transmission_interface/SimpleTransmission</type>
+            <joint name="${name}_${side}_drive_joint">
+                <hardwareInterface>hardware_interface/EffortJointInterface</hardwareInterface>
+            </joint>
+            <actuator name="${name}_${side}_drive_actuator}">
+                <mechanicalReduction>1</mechanicalReduction>
+            </actuator>
+        </transmission>
+        <transmission name="${name}_${side}_steer_transmission">
+            <type>transmission_interface/SimpleTransmission</type>
+            <joint name="${name}_${side}_steer_joint">
+                <hardwareInterface>hardware_interface/EffortJointInterface</hardwareInterface>
+            </joint>
+            <actuator name="${name}_${side}_steer_actuator">
+                <mechanicalReduction>1</mechanicalReduction>
+            </actuator>
+        </transmission>
     </xacro:macro>
 </robot>

Commit message: models update

File: urdf/rover.urdf.xacro (robot description, xacro)
@@ -5,6 +5,8 @@
 	<xacro:arg name="include_ros_control" default="true"/>
 	<xacro:arg name="realsense_use_nominal_extrinsics" default="true"/>
+	<xacro:arg name="show_cameras" default="true"/>
+	<xacro:arg name="show_laser_scan" default="true"/>
 	<!-- camera specific parameters -->
-	<xacro:arg name="topics_ns" default="Archimede"/>
+	<xacro:arg name="topics_ns" default="Archimede/d435i_camera"/>
 	<xacro:arg name="publish_pointcloud" default="true"/>
 	<xacro:arg name="add_plug" default="false"/>
@@ -35,5 +37,6 @@
 	</xacro:sensor_d435i>
 	<!-- Include Sensors -->
-	<xacro:rover_sensors name="Archimede"/>
+	<xacro:rover_sensors name="Archimede">
+	</xacro:rover_sensors>
 	<!-- Include Rover Plugins -->
 	<xacro:if value="$(arg include_plugins)">

File: urdf/xacros/plugins.xacro (robot description, xacro)
@@ -16,5 +16,19 @@
         </gazebo>
         <gazebo>
-            <plugin name="${name}_odometry_plugin" filename="libarchimede_odometry_gazebo_plugin.so"/>
+            <plugin name="${name}_odometry_plugin" filename="libarchimede_odometry_gazebo_plugin.so">
+                <!-- <topics_ns>Archimede<topics_ns/> -->
+                <integrator>Trapezi</integrator>
+                <odomTopicName>Archimede/odom</odomTopicName>
+                <odomQueSize>100</odomQueSize>
+                <odomFrameName>odom</odomFrameName>
+                <odomPublishRate>10</odomPublishRate>
+                <baseLinkFrameName>Archimede_foot_print</baseLinkFrameName>
+                <useFakePublishers>true</useFakePublishers>
+                <motorCurrentTopicName>Archimede/motor_current</motorCurrentTopicName>
+                <motorTemperatureTopicName>Archimede/motor_temperature</motorTemperatureTopicName>
+                <soundTopicName>Archimede/sound</soundTopicName>
+                <JointStateTopicName>Archimede/JointStateFake</JointStateTopicName>
+                <SensorStateTopicName>Archimede/sensor_state</SensorStateTopicName>
+            </plugin>
         </gazebo>
         <!-- INCLUDE HERE PLUGIN FOR IMU -->
@@ -51,4 +65,22 @@
                 <saveDir>$(find robot4ws_simulations)/data</saveDir>
                 <linkName>${name}_base_link</linkName>
+                <readCOG>false</readCOG>
+                <worldMode>true</worldMode>
+            </plugin>
+        </gazebo>
+        <gazebo>
+            <plugin name="${name}_get_fr_steer_hub_pose" filename="libarchimede_get_link_state.so">
+                <saveDir>$(find robot4ws_simulations)/data</saveDir>
+                <linkName>${name}_fr_steer_link</linkName>
+                <readCOG>false</readCOG>
+                <worldMode>false</worldMode>
+            </plugin>
+        </gazebo>
+        <gazebo>
+            <plugin name="${name}_magetic_sensor" filename="libhector_gazebo_ros_magnetic.so">
+                <updateRate>100</updateRate>
+                <robotNamespace>Archimede</robotNamespace>
+                <bodyName>${name}_imu_link</bodyName>
+                <topicName>magnetic_field</topicName>
             </plugin>
         </gazebo>

File: urdf/xacros/sensors.xacro (robot description, xacro)
@@ -28,6 +28,6 @@
                 </scan>
                 <range>
-                <min>0.2</min>
-                <max>3.5</max>
+                <min>1</min>
+                <max>5</max>
                 <resolution>0.015</resolution>
                 </range>

File: urdf/xacros/wheel_hub.xacro (robot description, xacro)
@@ -1,5 +1,5 @@
 <?xml version="1.0"?>
 <robot xmlns:xacro="http://www.ros.org/wiki/xacro" name="Archimede">
-	<xacro:macro name="rover_wheel_hub" params="name side reflect1 reflect2">
+	<xacro:macro name="rover_wheel_hub" params="name side reflect1 reflect2 use_simple_wheel:=true">
 		<xacro:property name="filename" value="$(find robot4ws_description)/urdf/config/wheel_hub.yaml"/>
 		<xacro:property name="wheel_config" value="${load_yaml (filename)}"/>
@@ -51,5 +51,5 @@
                     rpy="${data_tmp['orientation']['roll']} ${data_tmp['orientation']['pitch']} ${data_tmp['orientation']['yaw']}"/>
                     <geometry>
-                        <cylinder size="${wheel_config['drive']['geometry']['radius']} ${wheel_config['drive']['geometry']['length']}"/>
+                        <cylinder radius="${wheel_config['drive']['geom']['radius']}" length="${wheel_config['drive']['geom']['length']}"/>
                     </geometry>
                     <material name="gray"/>
@@ -58,5 +58,5 @@
             <collision>
                 <xacro:property name="data" value="${wheel_config['drive']['visual']}"/>
-                <xacro:if value="${data['mesh']}">
+                <xacro:unless value="${use_simple_wheel}">
                     <!-- Use mesh for visualization -->
                     <xacro:property name="data_tmp" value="${data['origin_mesh']}"/>
@@ -66,6 +66,6 @@
                         <mesh filename="package://robot4ws_description/meshes/${data['filename']}" scale="${data['mesh_scale']['x']} ${data['mesh_scale']['y']} ${data['mesh_scale']['z']}"/>
                     </geometry>
-                </xacro:if>
-                <xacro:unless value="${data['mesh']}">
+                </xacro:unless>
+                <xacro:if value="${use_simple_wheel}">
                     <!-- Use box as simple geometry visualization -->
                     <xacro:property name="data_tmp" value="${data['origin_simple_geom']}"/>
@@ -73,7 +73,22 @@
                     rpy="${data_tmp['orientation']['roll']} ${data_tmp['orientation']['pitch']} ${data_tmp['orientation']['yaw']}"/>
                     <geometry>
-                        <cylinder size="${wheel_config['drive']['geometry']['radius']} ${wheel_config['drive']['geometry']['length']}"/>
+                        <cylinder radius="${wheel_config['drive']['geom']['radius']}" length="${wheel_config['drive']['geom']['length']}"/>
                     </geometry>
-                </xacro:unless>
+                </xacro:if>
+                <surface>
+                    <friction>
+                    <ode>
+                        <mu>100.0</mu>
+                        <mu2>100.0</mu2>
+                    </ode>
+                    </friction>
+                    <contact>
+                    <ode>
+                        <kp>1e8</kp>
+                        <kd>1</kd>
+                        <min_depth>0.001</min_depth>
+                    </ode>
+                    </contact>
+                </surface>
             </collision>
         </link>
