Commit message: First stable commit

File: urdf/rover.urdf.xacro (robot description, xacro)
@@ -7,4 +7,5 @@
 	<xacro:arg name="show_cameras" default="true"/>
 	<xacro:arg name="show_laser_scan" default="true"/>
+	<xacro:arg name="rocker_differential" default="false"/>
 	<!-- camera specific parameters -->
 	<xacro:arg name="topics_ns" default="Archimede/d435i_camera"/>
@@ -12,4 +13,6 @@
 	<xacro:arg name="add_plug" default="false"/>
 	<xacro:include filename="$(find robot4ws_description)/urdf/xacros/rover_body.xacro"/>
+	<xacro:include filename="$(find robot4ws_description)/urdf/xacros/rover_differential.xacro"/>
+	<xacro:include filename="$(find robot4ws_description)/urdf/xacros/rover_leg.xacro"/>
 	<xacro:include filename="$(find robot4ws_description)/urdf/xacros/wheel_hub.xacro"/>
 	<xacro:include filename="$(find robot4ws_description)/urdf/xacros/materials.xacro"/>
@@ -18,17 +21,26 @@
 	<xacro:include filename="$(find realsense2_description)/urdf/_d435i.urdf.xacro"/>
 	<!-- Include rover base -->
-	<xacro:rover_base name="Archimede">
+	<xacro:rover_base name="Archimede" has_differential="$(arg rocker_differential)">
 	</xacro:rover_base>
+	<!-- Include legs if rocker_differential is flagged -->
+	<xacro:if value="$(arg rocker_differential)">
+		<xacro:rover_leg name="Archimede" reflect="1">
+		</xacro:rover_leg>
+		<xacro:rover_leg name="Archimede" reflect="-1">
+		</xacro:rover_leg>
+		<xacro:rover_differential name="Archimede">
+		</xacro:rover_differential>
+	</xacro:if>
 	<!-- Inlcude Front-Left wheel hub -->
-	<xacro:rover_wheel_hub name="Archimede" side="fl" reflect1="1" reflect2="1">
+	<xacro:rover_wheel_hub name="Archimede" side="fl" reflect1="1" reflect2="1" has_differential="$(arg rocker_differential)">
 	</xacro:rover_wheel_hub>
 	<!-- Include Back-Left wheel hub -->
-	<xacro:rover_wheel_hub name="Archimede" side="bl" reflect1="-1" reflect2="1">
+	<xacro:rover_wheel_hub name="Archimede" side="bl" reflect1="-1" reflect2="1" has_differential="$(arg rocker_differential)">
 	</xacro:rover_wheel_hub>
 	<!-- Include Back-Left wheel hub -->
-	<xacro:rover_wheel_hub name="Archimede" side="fr" reflect1="1" reflect2="-1">
+	<xacro:rover_wheel_hub name="Archimede" side="fr" reflect1="1" reflect2="-1" has_differential="$(arg rocker_differential)">
 	</xacro:rover_wheel_hub>
 	<!-- Include Back-Left wheel hub -->
-	<xacro:rover_wheel_hub name="Archimede" side="br" reflect1="-1" reflect2="-1">
+	<xacro:rover_wheel_hub name="Archimede" side="br" reflect1="-1" reflect2="-1" has_differential="$(arg rocker_differential)">
 	</xacro:rover_wheel_hub>
 	<!-- INCLUDE REALSENSE D435I STEREOCAMERA -->

File: urdf/xacros/plugins.xacro (robot description, xacro)
@@ -30,4 +30,6 @@
                 <JointStateTopicName>Archimede/JointStateFake</JointStateTopicName>
                 <SensorStateTopicName>Archimede/sensor_state</SensorStateTopicName>
+                <OdomMode>position</OdomMode>
+                <skipFrames>10</skipFrames>
             </plugin>
         </gazebo>

File: urdf/xacros/rover_body.xacro (robot description, xacro)
@@ -1,6 +1,14 @@
 <?xml version="1.0"?>
 <robot xmlns:xacro="http://www.ros.org/wiki/xacro" name="Archimede">
-	<xacro:macro name="rover_base" params="name">
-		<xacro:property name="filename" value="$(find robot4ws_description)/urdf/config/body.yaml"/>
+	<xacro:macro name="rover_base" params="name has_differential">
+		<!-- Depending whether the has_differential flag is on, select the correct yaml file -->
+		<xacro:if value="${has_differential}">
+			<xacro:property name="filename" value="$(find robot4ws_description)/urdf/config/body_only.yaml"/>
+			<xacro:property name="filenameTiltPlate" value="$(find robot4ws_description)/urdf/config/tilt_plate.yaml"/>
+			<xacro:property name="body_config_tiltPlate" value="${load_yaml (filenameTiltPlate)}"/>
+		</xacro:if>
+		<xacro:unless value="${has_differential}">
+			<xacro:property name="filename" value="$(find robot4ws_description)/urdf/config/body.yaml"/>
+		</xacro:unless>
 		<xacro:property name="body_config" value="${load_yaml (filename)}"/>
 		<!-- Define world link-->
@@ -38,4 +46,90 @@
 			</visual>
 		</link>
+		<!-- Tilt plate (only with differential) -->
+		<xacro:if value="${has_differential}">
+			<link name="${name}_tilt_plate">
+				<inertial>
+					<xacro:property name="data" value="${body_config_tiltPlate['body']['inertial']}"/>
+					<mass value="${data['mass']}"/>
+					<origin xyz="${data['origin']['position']['x']} ${data['origin']['position']['y']} ${data['origin']['position']['z']}"
+					rpy="${data['origin']['orientation']['roll']} ${data['origin']['orientation']['pitch']} ${data['origin']['orientation']['yaw']}"/>
+					<inertia ixx="${data['inertia']['ixx']}" ixy="${data['inertia']['ixy']}" ixz="${data['inertia']['ixz']}"
+				 	iyy="${data['inertia']['iyy']}" iyz="${data['inertia']['iyz']}" izz="${data['inertia']['izz']}"/>
+				</inertial>
+				<visual name="${name}_tilt_plate_visual">
+					<xacro:property name="data" value="${body_config_tiltPlate['body']['visual']}"/>
+					<xacro:if value="${data['mesh']}">
+						<!-- Use mesh for visualization -->
+						<xacro:property name="data_tmp" value="${data['origin_mesh']}"/>
+						<origin xyz="${data_tmp['position']['x']} ${data_tmp['position']['y']} ${data_tmp['position']['z']}"
+						rpy="${data_tmp['orientation']['roll']} ${data_tmp['orientation']['pitch']} ${data_tmp['orientation']['yaw']}"/>
+						<geometry>
+							<mesh filename="package://robot4ws_description/meshes/${data['filename']}" scale="${data['mesh_scale']['x']} ${data['mesh_scale']['y']} ${data['mesh_scale']['z']}"/>
+						</geometry>
+						<material name="black"/>
+					</xacro:if>
+					<xacro:unless value="${data['mesh']}">
+						<!-- Use box as simple geometry visualization -->
+						<xacro:property name="data_tmp" value="${data['origin_simple_geom']}"/>
+						<origin xyz="${data_tmp['position']['x']} ${data_tmp['position']['y']} ${data_tmp['position']['z']}"
+						rpy="${data_tmp['orientation']['roll']} ${data_tmp['orientation']['pitch']} ${data_tmp['orientation']['yaw']}"/>
+						<geometry>
+							<box size="${body_config_tiltPlate['body']['geometry']['body_length']} ${body_config_tiltPlate['body']['geometry']['body_width']} ${body_config_tiltPlate['body']['geometry']['body_heigth']}"/>
+						</geometry>
+					</xacro:unless>
+				</visual>
+			</link>
+		</xacro:if>
+		<!-- Define here the joint of the tilt plate to the body -->
+		<xacro:if value="${has_differential}">
+			<joint name="${name}_tilt_plate_joint" type="${body_config_tiltPlate['joint']['type']}">
+				<xacro:property name="tmp" value="${body_config_tiltPlate['joint']['origin']}"/>
+				<parent link="${name}_base_link_dummy"/>
+				<child link="${name}_tilt_plate"/>
+				<origin xyz="${tmp['position']['x']} ${tmp['position']['y']} ${tmp['position']['z']}"
+				rpy="${tmp['orientation']['roll']} ${tmp['orientation']['pitch']} ${tmp['orientation']['yaw']}"/>
+				<axis xyz="0 0 1"/>
+				<!-- <dynamic damping="0.1"/> -->
+			</joint>
+		</xacro:if>
+		<!-- Dummy joint link for the differential -->
+		<!-- <xacro:if value="${has_differential}">
+			<link name="${name}_dummy_disk">
+				<inertial>
+            		<origin xyz="0 0 0" rpy="0 0 0"/>
+					<mass value="1e-1"/>
+					<inertia ixx="1e-1" ixy="0" ixz="0" iyy="1e-1" iyz="0" izz="1e-1"/>
+				</inertial>
+				<visual>
+					Use disk as simple geometry visualization
+					<geometry>
+						<cylinder radius="0.05" length="0.05"/>
+						<box size="0.20 0.20 0.05"/>
+					</geometry>
+				</visual>
+			</link>
+		</xacro:if> -->
+		<!-- Define here the joint of the dummy disk -->
+		<!-- <xacro:if value="${has_differential}">
+			<joint name="${name}_dummy_joint" type="revolute">
+				<parent link="${name}_base_link_dummy"/>
+				<child link="${name}_dummy_disk"/>
+				<origin xyz="0 0 0" rpy="${-pi/2} 0 0"/>
+				<axis xyz="0 0 1"/>
+				<limit lower="0" upper="0" effort="1e6" velocity="1e6"/>
+			</joint>
+		</xacro:if> -->
+		<!-- <xacro:if value="${has_differential}">
+			<gazebo reference="{name}_dummy_joint">
+				<disableFixedJointLumping>true</disableFixedJointLumping>
+				<preserveFixedJoint>true</preserveFixedJoint>
+			</gazebo>
+		</xacro:if> -->
+		<!-- Define here the color of the dummy disk -->
+		<!-- <xacro:if value="${has_differential}">
+			<gazebo reference="${name}_dummy_disk">
+				<material>Gazebo/Blue</material>
+			</gazebo>
+		</xacro:if> -->
 		<!-- DEFINE HERE THE IMU LINK -->
 		<link name="${name}_imu_link"/>
@@ -80,4 +174,7 @@
 			<axis xyz="0 0 1"/>
 		</joint>
+		<!-- <gazebo reference="${name}_world_joint">
+			<preserveFixedJoint>false</preserveFixedJoint>
+		</gazebo> -->
 		<gazebo reference="${name}_base_link">
 			<material>Gazebo/Black</material>

File: urdf/xacros/wheel_hub.xacro (robot description, xacro)
@@ -1,7 +1,16 @@
 <?xml version="1.0"?>
-<robot xmlns:xacro="http://www.ros.org/wiki/xacro" name="Archimede">
-	<xacro:macro name="rover_wheel_hub" params="name side reflect1 reflect2 use_simple_wheel:=true">
+<robot xmlns:xacro="http://www.ros.org/wiki/xacro" name="Archimede" >
+    <xacro:arg name="point_contact" default="true"/>
+	<xacro:macro name="rover_wheel_hub" params="name side reflect1 reflect2 has_differential use_simple_wheel:=true">
 		<xacro:property name="filename" value="$(find robot4ws_description)/urdf/config/wheel_hub.yaml"/>
 		<xacro:property name="wheel_config" value="${load_yaml (filename)}"/>
+		<!-- Manage reflection -->
+        <!-- Get the legSide string (left/right) based on the value of reflect2 -->
+		<xacro:if value="${reflect2==1}">
+			<xacro:property name="legSide" value="left"/>
+		</xacro:if>
+		<xacro:if value="${reflect2==-1}">
+			<xacro:property name="legSide" value="right"/>
+		</xacro:if>
         <!-- Define here steer link-->
         <link name="${name}_${side}_steer_link">
@@ -17,7 +26,17 @@
         <joint name="${name}_${side}_steer_joint" type="${wheel_config['steer_joint']['type']}">
             <xacro:property name="tmp" value="${wheel_config['steer_joint']}"/>
-            <origin xyz="${reflect1*tmp['origin']['position']['x']} ${reflect2*tmp['origin']['position']['y']} ${tmp['origin']['position']['z']}"
-                rpy="${tmp['origin']['orientation']['roll']} ${tmp['origin']['orientation']['pitch']} ${tmp['origin']['orientation']['yaw']+(reflect2 -1)*pi/2}"/>
-            <parent link="${name}_base_link_dummy"/>
+            <!-- Manage the position of the wheels with respect to the model (with/without differential) -->
+            <!-- Without differential: wheel is attached to the body -->
+            <xacro:unless value="${has_differential}">
+                <origin xyz="${reflect1*tmp['origin']['position']['x']} ${reflect2*tmp['origin']['position']['y']} ${tmp['origin']['position']['z']}"
+                    rpy="${tmp['origin']['orientation']['roll']} ${tmp['origin']['orientation']['pitch']} ${tmp['origin']['orientation']['yaw']+(reflect2 -1)*pi/2}"/>
+                <parent link="${name}_base_link_dummy"/>
+            </xacro:unless>
+            <!-- With differential: wheel is attached to the leg -->
+            <xacro:if value="${has_differential}">
+                <origin xyz="${reflect1*tmp['origin']['position_withDifferential']['x']} ${reflect2*tmp['origin']['position_withDifferential']['y']} ${tmp['origin']['position_withDifferential']['z']}"
+                    rpy="${tmp['origin']['orientation']['roll']} ${tmp['origin']['orientation']['pitch']} ${tmp['origin']['orientation']['yaw']+(reflect2 -1)*pi/2}"/>
+                <parent link="${name}_leg_${legSide}"/>
+            </xacro:if>
             <child link="${name}_${side}_steer_link"/>
             <axis xyz="0 0 1"/>
@@ -72,21 +91,28 @@
                     <origin xyz="${data_tmp['position']['x']} ${data_tmp['position']['y']} ${data_tmp['position']['z']}"
                     rpy="${data_tmp['orientation']['roll']} ${data_tmp['orientation']['pitch']} ${data_tmp['orientation']['yaw']}"/>
-                    <geometry>
-                        <cylinder radius="${wheel_config['drive']['geom']['radius']}" length="${wheel_config['drive']['geom']['length']}"/>
-                    </geometry>
+                    <xacro:unless value="$(arg point_contact)">
+                        <geometry>
+                            <cylinder radius="${wheel_config['drive']['geom']['radius']}" length="0.001"/> <!-- "${wheel_config['drive']['geom']['length']}"/> -->
+                        </geometry>
+                    </xacro:unless>
+                    <xacro:if value="$(arg point_contact)">
+                        <geometry>
+                            <sphere radius="${wheel_config['drive']['geom']['radius']}"/>
+                        </geometry>
+                    </xacro:if>
                 </xacro:if>
                 <surface>
                     <friction>
-                    <ode>
-                        <mu>100.0</mu>
-                        <mu2>100.0</mu2>
-                    </ode>
+                        <ode>
+                            <!-- <mu>100.0</mu>
+                            <mu2>100.0</mu2> -->
+                        </ode>
                     </friction>
                     <contact>
-                    <ode>
-                        <kp>1e8</kp>
-                        <kd>1</kd>
-                        <min_depth>0.001</min_depth>
-                    </ode>
+                        <ode>
+                            <!-- <kp>1e8</kp>
+                            <kd>1</kd>
+                            <min_depth>0.001</min_depth> -->
+                        </ode>
                     </contact>
                 </surface>

Commit message: add velodyne lidar option

File: urdf/rover.urdf.xacro (robot description, xacro)
@@ -18,4 +18,7 @@
 	<xacro:arg name="publish_pointcloud" default="true"/>
 	<xacro:arg name="add_plug" default="false"/>
+	<!-- velodyne specific parameters -->
+	<xacro:arg name="add_velodyneHDL32E" default="false"/>
+	<xacro:arg name="lidar_organize_cloud" default="false"/>
 	<xacro:include filename="$(find robot4ws_description)/urdf/xacros/rover_body.xacro"/>
 	<xacro:include filename="$(find robot4ws_description)/urdf/xacros/rover_differential.xacro"/>
@@ -61,3 +64,10 @@
 		<xacro:rover_plugins name="Archimede" include_terrain_slip_plugin="$(arg include_terrain_slip_plugin)"/>
 	</xacro:if>
+	<!-- Include velodyne lidar -->
+	<xacro:if value="$(arg add_velodyneHDL32E)">
+		<xacro:include filename="$(find velodyne_description)/urdf/HDL-32E.urdf.xacro"/>
+		<xacro:HDL-32E parent="Archimede_base_link_dummy" name="Archimede_velodyne" topic="/Archimede/velodyne_points" organize_cloud="$(arg lidar_organize_cloud)" hz="10" samples="360">
+			<origin xyz="0.09 0 0.2" rpy="0 0 0" />
+		</xacro:HDL-32E>
+	</xacro:if>
 </robot>

Commit message: feat: add terramechanics model plugin

File: urdf/rover.urdf.xacro (robot description, xacro)
@@ -14,4 +14,5 @@
 	<xacro:arg name="rocker_differential" default="false"/>
 	<xacro:arg name="include_terrain_slip_plugin" default="true"/>
+	<xacro:arg name="include_wheels_terramechanic_model" default="false"/>
 	<!-- camera specific parameters -->
 	<xacro:arg name="topics_ns" default="Archimede/d435i_camera"/>
@@ -62,5 +63,5 @@
 	<!-- Include Rover Plugins -->
 	<xacro:if value="$(arg include_plugins)">
-		<xacro:rover_plugins name="Archimede" include_terrain_slip_plugin="$(arg include_terrain_slip_plugin)"/>
+		<xacro:rover_plugins name="Archimede" include_terrain_slip_plugin="$(arg include_terrain_slip_plugin)" include_wheels_terramechanic_model="$(arg include_wheels_terramechanic_model)"/>
 	</xacro:if>
 	<!-- Include velodyne lidar -->

File: urdf/xacros/plugins.xacro (robot description, xacro)
@@ -9,5 +9,5 @@
     <xacro:arg name="realsense_point_could" default="false"/>
     <!-- <xacro:arg name="" -->
-	<xacro:macro name="rover_plugins" params="name include_terrain_slip_plugin">
+	<xacro:macro name="rover_plugins" params="name include_terrain_slip_plugin include_wheels_terramechanic_model">
         <gazebo>
             <plugin name="gazebo_ros_control" filename="libgazebo_ros_control.so">
@@ -142,4 +142,25 @@
             </gazebo>
         </xacro:if>
+        <xacro:if value="${include_wheels_terramechanic_model}">
+            <xacro:property name="use_compact_model" value="true" /> <!-- true/false -->
+            <gazebo>
+                <plugin name="${name}_br_terramech_model" filename="libapply_single_wheel_terramechanic_model.so">
+                    <link_name>Archimede_br_wheel_link</link_name>
+                    <use_compact_model>${use_compact_model}</use_compact_model>
+                </plugin>
+                <plugin name="${name}_fr_terramech_model" filename="libapply_single_wheel_terramechanic_model.so">
+                    <link_name>Archimede_fr_wheel_link</link_name>
+                    <use_compact_model>${use_compact_model}</use_compact_model>
+                </plugin>
+                <plugin name="${name}_bl_terramech_model" filename="libapply_single_wheel_terramechanic_model.so">
+                    <link_name>Archimede_bl_wheel_link</link_name>
+                    <use_compact_model>${use_compact_model}</use_compact_model>
+                </plugin>
+                <plugin name="${name}_fl_terramech_model" filename="libapply_single_wheel_terramechanic_model.so">
+                    <link_name>Archimede_fl_wheel_link</link_name>
+                    <use_compact_model>${use_compact_model}</use_compact_model>
+                </plugin>
+            </gazebo>
+        </xacro:if>
 	</xacro:macro>
 </robot>
