Commit message: Feat: include gz_terramechanics plugin & new .world files

File: urdf/rover.urdf.xacro (robot description, xacro)
@@ -10,10 +10,11 @@
 	<xacro:arg name="include_ros_control" default="true"/>
 	<xacro:arg name="realsense_use_nominal_extrinsics" default="true"/>
-	<xacro:arg name="show_cameras" default="true"/>
-	<xacro:arg name="show_laser_scan" default="true"/>
+	<xacro:arg name="show_cameras" default="false"/>
+	<xacro:arg name="show_laser_scan" default="false"/>
 	<xacro:arg name="rocker_differential" default="false"/>
-	<xacro:arg name="include_terrain_slip_plugin" default="true"/>
+	<xacro:arg name="include_terrain_slip_plugin" default="false"/>
 	<xacro:arg name="include_wheels_terramechanic_model" default="false"/>
 	<xacro:arg name="load_sensors_plugins" default="true"/>
+	<xacro:arg name="terramechanics_config_path" default="/home/s250877/archimede_ros2_ws/src/archimede_rover/gz_terramechanics/config"/>
 	<!-- camera specific parameters -->
 	<xacro:arg name="topics_ns" default="Archimede/d435i_camera"/>
@@ -60,9 +61,9 @@
 	</xacro:sensor_d435i>
 	<!-- Include Sensors -->
-	<xacro:rover_sensors name="Archimede" add_velodyneHDL32E="$(arg add_velodyneHDL32E)">
+	<xacro:rover_sensors name="Archimede" add_velodyneHDL32E="$(arg add_velodyneHDL32E)" include_wheels_terramechanic_model="$(arg include_wheels_terramechanic_model)">
 	</xacro:rover_sensors>
 	<!-- Include Rover Plugins -->
 	<xacro:if value="$(arg include_plugins)">
-	<xacro:rover_plugins name="Archimede" include_terrain_slip_plugin="$(arg include_terrain_slip_plugin)" include_wheels_terramechanic_model="$(arg include_wheels_terramechanic_model)" load_sensors_plugins="$(arg load_sensors_plugins)"/>
+		<xacro:rover_plugins name="Archimede" include_terrain_slip_plugin="$(arg include_terrain_slip_plugin)" include_wheels_terramechanic_model="$(arg include_wheels_terramechanic_model)" load_sensors_plugins="$(arg load_sensors_plugins)" terramechanics_config_path="$(arg terramechanics_config_path)"/>
 	</xacro:if>
 	<!-- Include velodyne lidar -->

File: urdf/xacros/plugins.xacro (robot description, xacro)
@@ -1,8 +1,5 @@
 <?xml version="1.0"?>
 <robot xmlns:xacro="http://www.ros.org/wiki/xacro" name="Archimede">
-    <xacro:macro name="rover_plugins" params="name include_terrain_slip_plugin include_wheels_terramechanic_model load_sensors_plugins:=true">
-        <!-- Load wheel configuration from YAML, used in diff-drive/ackermann plugin - REMOVE -->
-        <!-- <xacro:property name="wheel_config_file" value="$(find robot4ws_description)/urdf/config/wheel_hub.yaml"/>
-        <xacro:property name="wheel_config" value="${xacro.load_yaml(wheel_config_file)}"/> -->
+    <xacro:macro name="rover_plugins" params="name include_terrain_slip_plugin include_wheels_terramechanic_model load_sensors_plugins:=true terramechanics_config_path">
         <gazebo>
             <plugin filename="gz-sim-joint-state-publisher-system"
@@ -25,40 +22,4 @@
                 <config_path>$(find robot4ws_gazebo_plugins)/config/joints_control_config.yaml</config_path>
             </plugin>
-            <!-- <plugin filename="gz-sim-diff-drive-system"
-                    name="gz::sim::systems::DiffDrive">
-                <left_joint>${name}_fl_drive_joint</left_joint>
-                <left_joint>${name}_bl_drive_joint</left_joint>
-                <right_joint>${name}_fr_drive_joint</right_joint>
-                <right_joint>${name}_br_drive_joint</right_joint>
-                <wheel_separation>${2 * wheel_config['steer_joint']['origin']['position']['y']}</wheel_separation>
-                <wheel_radius>${wheel_config['drive']['geom']['radius']}</wheel_radius>
-                <topic>cmd_vel</topic>
-                <odom_topic>odom</odom_topic>
-                <frame_id>odom</frame_id>
-                <child_frame_id>${name}_base_link</child_frame_id>
-            </plugin> -->
-            <!-- <plugin filename="gz-sim-ackermann-steering-system"
-                    name="gz::sim::systems::AckermannSteering">
-                <left_joint>${name}_fl_drive_joint</left_joint>
-                <left_joint>${name}_bl_drive_joint</left_joint>
-                <right_joint>${name}_fr_drive_joint</right_joint>
-                <right_joint>${name}_br_drive_joint</right_joint>
-                <left_steering_joint>${name}_fl_steer_joint</left_steering_joint>
-                <right_steering_joint>${name}_fr_steer_joint</right_steering_joint>
-                <wheel_base>${2 * wheel_config['steer_joint']['origin']['position']['x']}</wheel_base>
-                <wheel_separation>${2 * wheel_config['steer_joint']['origin']['position']['y']}</wheel_separation>
-                <wheel_radius>${wheel_config['drive']['geom']['radius']}</wheel_radius>
-                <steering_limit>0.5</steering_limit>
-                <min_velocity>-1</min_velocity>
-                <max_velocity>1</max_velocity>
-                <min_acceleration>-3</min_acceleration>
-                <max_acceleration>3</max_acceleration>
-                <topic>cmd_vel</topic>
-                <odom_topic>odom</odom_topic>
-                <frame_id>odom</frame_id>
-                <child_frame_id>${name}_base_link</child_frame_id>
-                <publish_odom>false</publish_odom>
-                <publish_tf>false</publish_tf>
-            </plugin> -->
         </gazebo>
         <gazebo>
@@ -70,5 +31,5 @@
                 <odom_covariance_topic>${name}/odom_with_covariance</odom_covariance_topic>
                 <tf_topic>tf</tf_topic>
-                <dimensions>2</dimensions>
+                <dimensions>3</dimensions>
                 <xyz_offset>0 0 0</xyz_offset>
                 <rpy_offset>0 0 0</rpy_offset>
@@ -76,5 +37,13 @@
             </plugin>
         </gazebo>
-        <!-- sensors remains: lidar, custom odometry -->
+        <!-- Terramechanics Plugin (optional) -->
+        <xacro:if value="${include_wheels_terramechanic_model}">
+            <gazebo>
+                <plugin filename="libTerramechanicsSystem.so" name="gz_terramechanics::TerramechanicsSystem">
+                    <config_path>${terramechanics_config_path}</config_path>
+                </plugin>
+            </gazebo>
+        </xacro:if>
+        <!-- sensors remains: lidar, custom odometry. These should be at .world file level -->
         <xacro:if value="${load_sensors_plugins}">
             <gazebo>

File: urdf/xacros/sensors.xacro (robot description, xacro)
@@ -11,5 +11,5 @@
     <xacro:arg name="visualize_scan" default="true"/>
     <xacro:arg name="visualize_lidar" default="true"/>
-	<xacro:macro name="rover_sensors" params="name add_velodyneHDL32E:=false">
+	<xacro:macro name="rover_sensors" params="name add_velodyneHDL32E:=false include_wheels_terramechanic_model">
     <!-- NOTE: the gz_frame_id block of each sensor will give a gazebo warning like this:
         [gz-2] Warning [Utils.cc:132] [/sdf/model[@name="Archimede"]/link[@name="Archimede_base_link"]/sensor[@name="rs_camera"]/gz_frame_id:<data-string>:L107]: XML Element[gz_frame_id], child of element[sensor], not defined in SDF. Copying[gz_frame_id] as children of [sensor].
@@ -166,4 +166,48 @@
             </gazebo>
         </xacro:if>
+        <!-- CONTACT SENSORS FOR TERRAMECHANICS PLUGIN -->
+        <!-- <xacro:if value="true"> -->
+        <xacro:if value="${include_wheels_terramechanic_model}">
+            <gazebo reference="Archimede_br_wheel_link">
+                <sensor name="Archimede_br_contact_sensor" type="contact">
+                    <contact>
+                        <collision>Archimede_br_wheel_link_collision</collision>
+                        <topic>${name}/br_contact_sensor</topic>
+                    </contact>
+                    <always_on>1</always_on>
+                    <update_rate>1000</update_rate>
+                </sensor>
+            </gazebo>
+            <gazebo reference="Archimede_fr_wheel_link">
+                <sensor name="Archimede_fr_contact_sensor" type="contact">
+                    <contact>
+                        <collision>Archimede_fr_wheel_link_collision</collision>
+                        <topic>${name}/fr_contact_sensor</topic>
+                    </contact>
+                    <always_on>1</always_on>
+                    <update_rate>1000</update_rate>
+                </sensor>
+            </gazebo>
+            <gazebo reference="Archimede_bl_wheel_link">
+                <sensor name="Archimede_bl_contact_sensor" type="contact">
+                    <contact>
+                        <collision>Archimede_bl_wheel_link_collision</collision>
+                        <topic>${name}/bl_contact_sensor</topic>
+                    </contact>
+                    <always_on>1</always_on>
+                    <update_rate>1000</update_rate>
+                </sensor>
+            </gazebo>
+            <gazebo reference="Archimede_fl_wheel_link">
+                <sensor name="Archimede_fl_contact_sensor" type="contact">
+                    <contact>
+                        <collision>Archimede_fl_wheel_link_collision</collision>
+                        <topic>${name}/fl_contact_sensor</topic>
+                    </contact>
+                    <always_on>1</always_on>
+                    <update_rate>1000</update_rate>
+                </sensor>
+            </gazebo>
+        </xacro:if>
     </xacro:macro>
 </robot>

File: urdf/xacros/wheel_hub.xacro (robot description, xacro)
@@ -107,19 +107,4 @@
                     </xacro:if>
                 </xacro:if>
-                <surface>
-                    <friction>
-                        <ode>
-                            <!-- <mu>100.0</mu>
-                            <mu2>100.0</mu2> -->
-                        </ode>
-                    </friction>
-                    <contact>
-                        <ode>
-                            <!-- <kp>1e8</kp>
-                            <kd>1</kd>
-                            <min_depth>0.001</min_depth> -->
-                        </ode>
-                    </contact>
-                </surface>
             </collision>
         </link>
